File: schematic/schematic.kicad_sch (KiCad schematic)
At the start: 0 parts

Commit message: Progress on KiCAD schematics
Other:
- title: Da Vinci Jr. 1.0 schematic -> (none)
Changed lines of the file:
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@@
 	(generator_version "10.0")
 	(paper "A4")
-	(title_block
-		(title "Da Vinci Jr. 1.0 schematic")
-		(date "2026-08-26")
-		(rev "1")
-		(comment 1 "The main schematic for the printer, its used for organizing all the other board files etc")
-	)
 	(sheet
-		(at 203.2 30.48)
-		(size 67.31 120.65)
+		(at 157.48 36.83)
+		(size 62.23 58.42)
 		(exclude_from_sim no)
 		(in_bom yes)
@@
 		)
 		(property "Sheetname" "Sub Board"
-			(at 203.2 29.7684 0)
+			(at 157.48 36.1184 0)
 			(show_name no)
 			(do_not_autoplace no)
@@
 		)
 		(property "Sheetfile" "SubBoard.kicad_sch"
-			(at 203.2 151.7146 0)
+			(at 157.48 95.8346 0)
 			(show_name no)
 			(do_not_autoplace no)
@@
 		)
 		(instances
-			(project "DaVinciJr1.0"
+			(project "schematic"
 				(path "/1e12c736-bef9-40e8-b505-1000ff77a2bb"
-					(page "3")
+					(page "1")
 				)
 			)
@@
 	)
 	(sheet
-		(at 20.32 29.21)
-		(size 161.29 106.68)
+		(at 20.32 22.86)
+		(size 52.07 55.88)
 		(exclude_from_sim no)
 		(in_bom yes)
@@
 		)
 		(property "Sheetname" "Main Board"
-			(at 20.32 28.4984 0)
+			(at 20.32 22.1484 0)
 			(show_name no)
 			(do_not_autoplace no)
@@
 		)
 		(property "Sheetfile" "MainBoard.kicad_sch"
-			(at 20.32 136.4746 0)
+			(at 20.32 79.3246 0)
 			(show_name no)
 			(do_not_autoplace no)
@@
 		)
 		(instances
-			(project "DaVinciJr1.0"
+			(project "schematic"
 				(path "/1e12c736-bef9-40e8-b505-1000ff77a2bb"
-					(page "2")
+					(page "1")
 				)
 			)
@@
 	)
 	(sheet
-		(at 38.1 144.78)
-		(size 77.47 40.64)
+		(at 67.31 123.19)
+		(size 50.8 40.64)
 		(exclude_from_sim no)
 		(in_bom yes)
@@
 		)
 		(property "Sheetname" "Hotend Board"
-			(at 38.1 144.0684 0)
+			(at 67.31 122.4784 0)
 			(show_name no)
 			(do_not_autoplace no)
@@
 		)
 		(property "Sheetfile" "HotendBoard.kicad_sch"
-			(at 38.1 186.0046 0)
+			(at 67.31 164.4146 0)
 			(show_name no)
 			(do_not_autoplace no)
@@
 		)
 		(instances
-			(project "DaVinciJr1.0"
+			(project "schematic"
 				(path "/1e12c736-bef9-40e8-b505-1000ff77a2bb"
-					(page "4")
+					(page "1")
 				)
 			)
