File: schematic/MainBoard.kicad_sch (KiCad schematic)
At the start: 0 parts

Commit message: Progress on KiCAD schematics
Parts:
- added U1: LPC1115FBD48-303, Package_QFP:LQFP-48_7x7mm_P0.5mm, symbol MCU_NXP_LPC:LPC1115FBD48-303
Other:
- title: (none) -> Da Vinci Jr. 1.0 Main Board schematic
Changed lines of the file:
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@@
 	(generator_version "10.0")
 	(paper "A4")
+	(title_block
+		(title "Da Vinci Jr. 1.0 Main Board schematic")
+		(date "2026-08-26")
+		(rev "1")
+	)
+	(symbol
+		(lib_id "MCU_NXP_LPC:LPC1115FBD48-303")
+		(at 224.79 73.66 0)
+		(unit 1)
+		(body_style 1)
+		(exclude_from_sim no)
+		(in_bom yes)
+		(on_board yes)
+		(in_pos_files yes)
+		(dnp no)
+		(fields_autoplaced yes)
+		(property "Reference" "U1"
+			(at 229.4733 34.29 0)
+			(show_name no)
+			(do_not_autoplace no)
+			(effects
+				(font
+					(size 1.27 1.27)
+				)
+				(justify left)
+			)
+		)
+		(property "Value" "LPC1115FBD48-303"
+			(at 229.4733 36.83 0)
+			(show_name no)
+			(do_not_autoplace no)
+			(effects
+				(font
+					(size 1.27 1.27)
+				)
+				(justify left)
+			)
+		)
+		(property "Footprint" "Package_QFP:LQFP-48_7x7mm_P0.5mm"
+			(at 247.65 35.56 0)
+			(hide yes)
+			(show_name no)
+			(do_not_autoplace no)
+			(effects
+				(font
+					(size 1.27 1.27)
+				)
+			)
+		)
+		(property "Datasheet" "http://www.nxp.com/docs/en/data-sheet/LPC111X.pdf"
+			(at 273.05 58.42 0)
+			(hide yes)
+			(show_name no)
+			(do_not_autoplace no)
+			(effects
+				(font
+					(size 1.27 1.27)
+				)
+			)
+		)
+		(property "Description" "32-bit ARM Cortex-M0 microcontroller, 64KB flash, 8KB SRAM, power profile"
+			(at 224.79 73.66 0)
+			(hide yes)
+			(show_name no)
+			(do_not_autoplace no)
+			(effects
+				(font
+					(size 1.27 1.27)
+				)
+			)
+		)
+		(pin "14"
+		)
+		(pin "8"
+		)
+		(pin "7"
+		)
+		(pin "9"
+		)
+		(pin "6"
+		)
+		(pin "5"
+		)
+		(pin "13"
+		)
+		(pin "4"
+		)
+		(pin "12"
+		)
+		(pin "11"
+		)
+		(pin "10"
+		)
+		(pin "3"
+		)
+		(pin "17"
+		)
+		(pin "16"
+		)
+		(pin "24"
+		)
+		(pin "25"
+		)
+		(pin "15"
+		)
+		(pin "20"
+		)
+		(pin "26"
+		)
+		(pin "19"
+		)
+		(pin "22"
+		)
+		(pin "18"
+		)
+		(pin "23"
+		)
+		(pin "21"
+		)
+		(pin "2"
+		)
+		(pin "36"
+		)
+		(pin "35"
+		)
+		(pin "34"
+		)
+		(pin "33"
+		)
+		(pin "32"
+		)
+		(pin "31"
+		)
+		(pin "30"
+		)
+		(pin "29"
+		)
+		(pin "28"
+		)
+		(pin "27"
+		)
+		(pin "47"
+		)
+		(pin "46"
+		)
+		(pin "45"
+		)
+		(pin "44"
+		)
+		(pin "43"
+		)
+		(pin "42"
+		)
+		(pin "41"
+		)
+		(pin "48"
+		)
+		(pin "40"
+		)
+		(pin "38"
+		)
+		(pin "39"
+		)
+		(pin "37"
+		)
+		(pin "1"
+		)
+		(instances
+			(project "DaVinciJr1.0"
+				(path "/1e12c736-bef9-40e8-b505-1000ff77a2bb/d610c2e8-63cd-4e0f-98e2-bf1a99df609b"
+					(reference "U1")
+					(unit 1)
+				)
+			)
+		)
+	)
 )

Commit message: Update board schematics
Parts:
- renumbered U1 to U17
Other:
- moved on the sheet: U17
Changed lines of the file:
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@@
 	(symbol
 		(lib_id "MCU_NXP_LPC:LPC1115FBD48-303")
-		(at 224.79 73.66 0)
+		(at 219.71 76.2 0)
 		(unit 1)
 		(body_style 1)
@@
 		(dnp no)
 		(fields_autoplaced yes)
-		(property "Reference" "U1"
-			(at 229.4733 34.29 0)
+		(property "Reference" "U17"
+			(at 224.3933 36.83 0)
 			(show_name no)
 			(do_not_autoplace no)
@@
 		)
 		(property "Value" "LPC1115FBD48-303"
-			(at 229.4733 36.83 0)
+			(at 224.3933 39.37 0)
 			(show_name no)
 			(do_not_autoplace no)
@@
 		)
 		(property "Footprint" "Package_QFP:LQFP-48_7x7mm_P0.5mm"
-			(at 247.65 35.56 0)
+			(at 242.57 38.1 0)
 			(hide yes)
 			(show_name no)
@@
 		)
 		(property "Datasheet" "http://www.nxp.com/docs/en/data-sheet/LPC111X.pdf"
-			(at 273.05 58.42 0)
+			(at 267.97 60.96 0)
 			(hide yes)
 			(show_name no)
@@
 		)
 		(property "Description" "32-bit ARM Cortex-M0 microcontroller, 64KB flash, 8KB SRAM, power profile"
-			(at 224.79 73.66 0)
+			(at 219.71 76.2 0)
 			(hide yes)
 			(show_name no)
@@
 			(project "DaVinciJr1.0"
 				(path "/1e12c736-bef9-40e8-b505-1000ff77a2bb/d610c2e8-63cd-4e0f-98e2-bf1a99df609b"
-					(reference "U1")
+					(reference "U17")
 					(unit 1)
 				)

Commit message: Start main board schematic and update hotend schematic size
Parts:
- added J1, J12, J13, J4, J5: Conn_01x04_Pin, symbol Connector:Conn_01x04_Pin
- added J11: Conn_02x06_Row_Letter_First, symbol Connector_Generic:Conn_02x06_Row_Letter_First
- added J14: Conn_01x03_Pin, symbol Connector:Conn_01x03_Pin
- added J15: Conn_01x02_Pin, symbol Connector:Conn_01x02_Pin
- added J16: Conn_01x06_Pin, symbol Connector:Conn_01x06_Pin
- added J17: USB_B, symbol Connector:USB_B
- added J18: Jack-DC, symbol Connector:Jack-DC
- added SW7: SW_DPST_x2, symbol Switch:SW_DPST_x2
- added U2: ATSAM4E8EA-AU, LQFP144_ATM, symbol 2026-08-26_20-46-55:ATSAM4E8EA-AU
- added U3: MX25L3206E, Package_SO:SOIC-8_5.3x5.3mm_P1.27mm, symbol Memory_Flash:MX25L3233FM2
- added U4, U6, U7, U8: TB62269FTG, Package_QFP:LQFP-48_7x7mm_P0.5mm, symbol TB62269FTG:TB62269FTG
Other:
- moved on the sheet: U17

Commit message: Updata TODO and schematics
Parts:
- removed J11: Conn_02x06_Row_Letter_First, symbol Connector_Generic:Conn_02x06_Row_Letter_First
- removed J15: Conn_01x02_Pin, symbol Connector:Conn_01x02_Pin
- removed J16: Conn_01x06_Pin, symbol Connector:Conn_01x06_Pin
- removed SW7: SW_DPST_x2, symbol Switch:SW_DPST_x2
- added J12-J123: NFC, symbol Connector_Generic:Conn_02x06_Row_Letter_First
- added J121-J122: Reflow FAN, symbol Connector:Conn_01x04_Pin
- added J37: Home Sensor, symbol Connector_Generic:Conn_02x06_Counter_Clockwise
- added R217: 1M, Resistor_THT:R_Axial_DIN0207_L6.3mm_D2.5mm_P10.16mm_Horizontal, symbol PCM_SL_Resistors:1M
- added R291: Unknown, Resistor_THT:R_Axial_DIN0207_L6.3mm_D2.5mm_P10.16mm_Horizontal, symbol PCM_SL_Resistors:Resistor
- added SW5: Rocker, symbol Switch:SW_SPDT
- J19-J14: renamed from J1; value Conn_01x04_Pin -> Pull Filament
- J29: renamed from J12; value Conn_01x04_Pin -> Motor-E1
- J35: renamed from J18; value Jack-DC -> Adaptor
Connections:
- net at J29.1 (Pin_1): now also U8.10 (OUT_A1), U8.11 (OUT_A2)
- net at J29.2 (Pin_2): now also U8.16 (OUT_A1-), U8.17 (OUT_A2-)
- net at J29.3 (Pin_3): now also U8.20 (OUT_B2-), U8.21 (OUT_B1-)
- net at J29.4 (Pin_4): now also U8.26 (OUT_B2), U8.27 (OUT_B1)
- net at J35.1: now also SW5.1 (A)
- net GNDREF: now reaches J35.2
- net GNDREF: now also J17.4 (GND), J19-J14.3 (Pin_3), U8.15 (GND), U8.18 (GND), U8.19 (GND), U8.22 (GND), R217.2
- net +3.3V: now reaches J19-J14.4 (Pin_4)
- net at J17.SH (Shield): now also R217.1
- new net: J121-J122.2 (Pin_2), J121-J122.3 (Pin_3), R291.2
- new net +12V: R291.1, SW5.2 (B)

Commit message: Document SAM4E pinouts and update schematic
Parts:
- J25: renamed from J5; value Conn_01x04_Pin -> Motor-X
- J26: renamed from J4; value Conn_01x04_Pin -> Motor-Y
- J27: renamed from J13; value Conn_01x04_Pin -> Motor-Z
- renumbered U4 to U10, U6 to U11, U7 to U12, U8 to U14
Connections:
- net GNDREF: now also U10.15 (GND), U10.18 (GND), U10.19 (GND), U10.22 (GND), U10.5 (GND), U11.15 (GND), U11.18 (GND), U11.19 (GND), U11.5 (GND), U12.15 (GND), U12.18 (GND), U12.19 (GND), U12.22 (GND), U12.5 (GND), U14.5 (GND)
- net at U10.10 (OUT_A1): now also J25.1 (Pin_1), U10.11 (OUT_A2)
- net at U10.16 (OUT_A1-): now also J25.2 (Pin_2), U10.17 (OUT_A2-)
- net at U10.2 (CLK_IN): now also U2.127 (PC23)
- net at U10.20 (OUT_B2-): now also J25.3 (Pin_3), U10.21 (OUT_B1-)
- net at U10.26 (OUT_B2): now also J25.4 (Pin_4), U10.27 (OUT_B1)
- net at U10.3 (ENABLE): now also U2.128 (PD3)
- net at U10.44 (CW/CCW): now also U2.126 (PD4)
- net at U2.119 (PD7): now also U12.44 (CW/CCW)
- net at U2.120 (PC20): now also U12.2 (CLK_IN)
- net at U2.121 (PD6): now also U12.3 (ENABLE)
- net at U2.124 (PC22): now also U11.2 (CLK_IN)
- net at U2.125 (PD5): now also U11.3 (ENABLE)
- net at U2.74 (PD17): now also U14.44 (CW/CCW)
- net at U2.76 (PC28): now also U14.2 (CLK_IN)
- net at U2.78 (PD16): now also U14.3 (ENABLE)
- net at U11.10 (OUT_A1): now also J26.1 (Pin_1), U11.11 (OUT_A2)
- net at U11.16 (OUT_A1-): now also J26.2 (Pin_2), U11.17 (OUT_A2-)
- net at U11.20 (OUT_B2-): now also J26.3 (Pin_3), U11.21 (OUT_B1-)
- net at U11.26 (OUT_B2): now also J26.4 (Pin_4), U11.27 (OUT_B1)
- net at U11.44 (CW/CCW): now also U2.7 (PE2)
- net at J27.1 (Pin_1): now also U12.10 (OUT_A1), U12.11 (OUT_A2)
- net at J27.2 (Pin_2): now also U12.16 (OUT_A1-), U12.17 (OUT_A2-)
- net at J27.3 (Pin_3): now also U12.20 (OUT_B2-), U12.21 (OUT_B1-)
- net at J27.4 (Pin_4): now also U12.26 (OUT_B2), U12.27 (OUT_B1)
- no-connect marks 0 -> 16
Other:
- moved on the sheet: J19-J14, J25

Commit message: Document board power fuses and update power schematics
Parts:
- added C192, C217, C218, C222, C223, C224, C233, C234: (no value), symbol Device:C_Small
- added C24, C30: Capacitor, symbol Device:C_Small
- added D1, D2: LED, symbol Device:LED
- added F1, R293: Fuse, symbol Device:Fuse
- added L27: 150, symbol Device:L
- added L28: 100, symbol Device:L
- added R140: 0.2, symbol Device:R
- added R2: 560, Resistor_THT:R_Axial_DIN0207_L6.3mm_D2.5mm_P10.16mm_Horizontal, symbol PCM_SL_Resistors:100k
- added R247, R282, R283: 10k, Resistor_THT:R_Axial_DIN0207_L6.3mm_D2.5mm_P10.16mm_Horizontal, symbol PCM_SL_Resistors:12k
- added R280: 20k, Resistor_THT:R_Axial_DIN0207_L6.3mm_D2.5mm_P10.16mm_Horizontal, symbol PCM_SL_Resistors:12k
- added R281, R285: 100k, Resistor_THT:R_Axial_DIN0207_L6.3mm_D2.5mm_P10.16mm_Horizontal, symbol PCM_SL_Resistors:100k
- added R284: 12k, Resistor_THT:R_Axial_DIN0207_L6.3mm_D2.5mm_P10.16mm_Horizontal, symbol PCM_SL_Resistors:12k
- added R3: 1k, Resistor_THT:R_Axial_DIN0207_L6.3mm_D2.5mm_P10.16mm_Horizontal, symbol PCM_SL_Resistors:100k
- added R305: 10k, Resistor_THT:R_Axial_DIN0207_L6.3mm_D2.5mm_P10.16mm_Horizontal, symbol PCM_SL_Resistors:10k
- added RV25, RV26: Varistor, symbol Device:Varistor
- added U21, U22: RT7248H, Package_DFN_QFN:Texas_RGW0020A_VQFN-20-1EP_5x5mm_P0.65mm_EP3.15x3.15mm_ThermalVias, symbol Regulator_Linear:TPS7A3301RGW
- added Y1: Crystal_12MHz, Crystal:Crystal_HC49-4H_Vertical, symbol PCM_SL_Devices:Crystal_16MHz
Connections:
- net +12V: now also R293.1
- net GNDREF: now also C218.1, C224.2, C233.1, C234.2, C24.1, C30.1, D1.1 (K), D2.1 (K), R247.2, R280.2, R282.2, R284.2, R305.1, RV25.2, RV26.2
- net at U2.141 (PB8): now also C24.2, Y1.2
- net at U2.142 (PB9): now also C30.2, Y1.1
- net at J17.2 (D-): now also RV25.1
- net at J17.3 (D+): now also RV26.1
- net at U12.4 (RESET): now also R305.2
- net at U12.7 (RS_A1): now also U12.8 (RS_A2), R140.2
- new net: R247.1, U21.5 (FB)
- new net: C218.2, C233.2, U21.8 (SS)
- new net: C222.1, U22.1 (BOOT)
- new net: C222.2, L28.1, U22.3 (SW)
- new net: R281.2, R285.2, R293.2, U21.2 (VIN), U22.2 (VIN)
- new net: C217.1, U21.6 (COMP)
- new net: C217.2, R280.1
- new net: D1.2 (A), R2.2
- new net: R281.1, U21.7 (EN)
- new net: R282.1, R283.1, U22.5 (FB)
- new net: L28.2, R2.1, R283.2
- new net: D2.2 (A), R3.2
- new net: C223.1, U21.4 (GND), U22.4 (GND), U22.6 (COMP)
- new net: R285.1, U22.7 (EN)
- new net: C224.1, C234.1, U22.8 (SS)
- new net: L27.2, R3.1
- new net: C223.2, R284.1
- new net: C192.1, U21.1 (BOOT)
- new net: C192.2, L27.1, U21.3 (SW)
- no-connect marks 16 -> 32
Other:
- moved on the sheet: J14, J29

Commit message: Complete hotend documentation and schematics
Other:
- moved on the sheet: C192, C217, C218, C222, C223, C224, C233, C234, C24, C30, D1, D2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
