File: schematic/MainBoard.kicad_sch (KiCad schematic)
At the start: 53 parts, among them J12-J123 NFC, J121-J122 Reflow FAN, J14 Conn_01x03_Pin, J17 USB_B, J19-J14 Pull Filament, J25 Motor-X, J26 Motor-Y, J27 Motor-Z, J29 Motor-E1, J35 Adaptor, J37 Home Sensor, SW5 Rocker, U10 TB62269FTG, U11 TB62269FTG, U12 TB62269FTG, U14 TB62269FTG, U17 LPC1115FBD48-303, U2 ATSAM4E8EA-AU, U21 RT7248H, U22 RT7248H, U3 MX25L3206E, Y1 Crystal_12MHz

Commit message: Update main board schematic
Parts:
- added BZ1: AC-1203D-RP, Buzzer_Beeper:MagneticBuzzer_ProSignal_ABT-410-RC, symbol PCM_SL_Devices:Buzzer_5V
- added J6: Conn_02x08_Odd_Even, symbol Connector_Generic:Conn_02x08_Odd_Even
- added J7: Conn_02x11_Odd_Even, symbol Connector_Generic:Conn_02x11_Odd_Even
- added J8: Conn_01x51_Pin, symbol Connector:Conn_01x51_Pin
- J5: renamed from J14; value Conn_01x03_Pin -> TopLamp
Connections:
- net at J25.1 (Pin_1), U10.10 (OUT_A1), U10.11 (OUT_A2): now also J25.3 (Pin_3), U10.20 (OUT_B2-), U10.21 (OUT_B1-)
- no-connect marks 32 -> 64
Other:
- moved on the sheet: C24, C30, J12-J123, J19-J14, J25, J26, J27, J29, J37, J5, R140, R305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

Commit message: Update schematic for the drivers power rails
Parts:
- removed R291: Unknown, Resistor_THT:R_Axial_DIN0207_L6.3mm_D2.5mm_P10.16mm_Horizontal, symbol PCM_SL_Resistors:Resistor
- added Q3: PMBT2222A, Package_TO_SOT_SMD:SOT-23, symbol Transistor_BJT:PMBT2222A
- added Q8: TPC8067, Package_TO_SOT_SMD:LFPAK33, symbol Transistor_FET:BUK7M27-80EX
- added R105, R106, R120, R121, R131, R164, R176: 0.2, symbol Device:R
- added R279, R291: Fuse, symbol Device:Fuse
- added R303, R304, R307: 10k, Resistor_THT:R_Axial_DIN0207_L6.3mm_D2.5mm_P10.16mm_Horizontal, symbol PCM_SL_Resistors:10k
- J8: value Conn_01x51_Pin -> Nozz/FAN/NTC/SW
- renumbered F1 to R292
Connections:
- net +12V: now also R292.1, R279.1, R291.1
- net GNDREF: now also Q8.1 (S), Q8.2 (S), Q8.3 (S), R303.1, R304.1, R307.1
- net at J8.1 (Pin_1): now also J8.2 (Pin_2), J8.3 (Pin_3), J8.4 (Pin_4), J8.46 (Pin_46), J8.47 (Pin_47), J8.48 (Pin_48), J8.49 (Pin_49), J8.5 (Pin_5), J8.50 (Pin_50), J8.51 (Pin_51), J8.6 (Pin_6), R292.2
- net at J8.10 (Pin_10): now also J8.11 (Pin_11), J8.12 (Pin_12), J8.13 (Pin_13), J8.14 (Pin_14), J8.38 (Pin_38), J8.39 (Pin_39), J8.40 (Pin_40), J8.41 (Pin_41), J8.42 (Pin_42), J8.43 (Pin_43), J8.9 (Pin_9), Q8.5 (D)
- net at J25.1 (Pin_1), U10.10 (OUT_A1), U10.11 (OUT_A2): no longer J25.3 (Pin_3), U10.20 (OUT_B2-), U10.21 (OUT_B1-)
- net at U10.29 (RS_B2): now also U10.30 (RS_B1), R105.1
- net at U10.4 (RESET): now also R303.2
- net at U10.7 (RS_A1): now also U10.8 (RS_A2), R120.1
- net at U11.29 (RS_B2): now also U11.30 (RS_B1), R106.1
- net at U11.4 (RESET): now also R304.2
- net at U11.7 (RS_A1): now also U11.8 (RS_A2), R121.1
- net at R140.1: now also U12.7 (RS_A1), U12.8 (RS_A2)
- net at J121-J122.2 (Pin_2), J121-J122.3 (Pin_3): now also R291.2
- net at U14.29 (RS_B2): now also U14.30 (RS_B1), R164.1
- net at U14.4 (RESET): now also R307.2
- net at U14.7 (RS_A1): now also U14.8 (RS_A2), R176.1
- net at U12.29 (RS_B2): now also U12.30 (RS_B1), R131.1
- new net: R105.2, R106.2, R120.2, R121.2, R131.2, R140.2, R164.2, R176.2, R279.2
- new net: J25.3 (Pin_3), U10.20 (OUT_B2-), U10.21 (OUT_B1-)
- no-connect marks 64 -> 72
Other:
- moved on the sheet: J17, J25, J8, R140, R217, R292, R293, RV25, RV26

Commit message: Update schematic and progress, verify some pins
Parts:
- J6: renamed from J7; value Conn_02x11_Odd_Even -> LCM
- SD1: renamed from J6; value Conn_02x08_Odd_Even -> SD
Connections:
- net +3.3V: now also L28.2, R2.1, R283.2
- net GNDREF: now also J5.2 (Pin_2), SD1.2 (Pin_2), SD1.4 (Pin_4), SD1.6 (Pin_6)
- net at R105.2, R106.2, R120.2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: now also J5.3 (Pin_3)
- net +5V: now reaches L27.2, R3.1
